Commit message: working walking gaitgit add -A :/git add -A :/

File: laikago/laikago.urdf (robot description, URDF)
Before this commit: robot plane, 13 links, 12 joints
Links:
- link FL_hip_motor: geometry collision mesh filename=package://jelly_locomotion/laikago/hip_motor.stl scale=1 1 1; visual mesh filename=package://jelly_locomotion/laikago/hip_motor.stl scale=1 1 1
- link FL_lower_leg: geometry collision mesh filename=package://jelly_locomotion/laikago/lower_leg_3.stl scale=1 1 1; visual mesh filename=package://jelly_locomotion/laikago/lower_leg_3.stl scale=1 1 1
- link FL_upper_leg: geometry collision mesh filename=package://jelly_locomotion/laikago/upper_leg_left_vhacd.obj scale=1 1 1; visual mesh filename=package://jelly_locomotion/laikago/upper_leg.stl scale=1 1 1
- link FR_hip_motor: geometry collision mesh filename=package://jelly_locomotion/laikago/hip_motor_mirror.stl scale=1 1 1; visual mesh filename=package://jelly_locomotion/laikago/hip_motor_mirror.stl scale=1 1 1
- link FR_lower_leg: geometry collision mesh filename=package://jelly_locomotion/laikago/lower_leg_3.stl scale=1 1 1; visual mesh filename=package://jelly_locomotion/laikago/lower_leg_3.stl scale=1 1 1
- link FR_upper_leg: geometry collision mesh filename=package://jelly_locomotion/laikago/upper_leg_right_vhacd.obj scale=1 1 1; visual mesh filename=package://jelly_locomotion/laikago/upper_leg_mirror.stl scale=1 1 1
- link RL_hip_motor: geometry collision mesh filename=package://jelly_locomotion/laikago/hip_motor.stl scale=1 1 1; visual mesh filename=package://jelly_locomotion/laikago/hip_motor.stl scale=1 1 1
- link RL_lower_leg: geometry collision mesh filename=package://jelly_locomotion/laikago/lower_leg_3.stl scale=1 1 1; visual mesh filename=package://jelly_locomotion/laikago/lower_leg_3.stl scale=1 1 1
- link RL_upper_leg: geometry collision mesh filename=package://jelly_locomotion/laikago/upper_leg_left_vhacd.obj scale=1 1 1; visual mesh filename=package://jelly_locomotion/laikago/upper_leg.stl scale=1 1 1
- link RR_hip_motor: geometry collision mesh filename=package://jelly_locomotion/laikago/hip_motor_mirror.stl scale=1 1 1; visual mesh filename=package://jelly_locomotion/laikago/hip_motor_mirror.stl scale=1 1 1
- link RR_lower_leg: geometry collision mesh filename=package://jelly_locomotion/laikago/lower_leg_3.stl scale=1 1 1; visual mesh filename=package://jelly_locomotion/laikago/lower_leg_3.stl scale=1 1 1
- link RR_upper_leg: geometry collision mesh filename=package://jelly_locomotion/laikago/upper_leg_right_vhacd.obj scale=1 1 1; visual mesh filename=package://jelly_locomotion/laikago/upper_leg_mirror.stl scale=1 1 1
- link chassis: geometry collision mesh filename=package://jelly_locomotion/laikago/chassis_vhacd_mod.obj scale=1 1 1; visual mesh filename=package://jelly_locomotion/laikago/chassis.stl scale=1 1 1
