Commit message: fixed ik, working on gaits

File: scripts/data/jelly/jelly.urdf (robot description, URDF)
Before this commit: robot jelly_description, 13 links, 12 joints
Links:
- link base_link: mass 1.4036 -> 2.4036
Joints:
- joint FL_hip_joint: axis 1 0 0 -> -1 0 0
- joint RL_hip_joint: axis 1 0 0 -> -1 0 0

Commit message: for travis

File: scripts/data/jelly/jelly.urdf (robot description, URDF)
Before this commit: robot jelly_description, 13 links, 12 joints
Links:
- link base_link: mass 2.4036 -> 5.4036
